File: WaveKitty/WKController/WKController/WKController.kicad_pcb (KiCad board)
At the start: 2 copper layers, 88.3 x 38.1 mm, 15 parts, among them J1 MIDI, J2 Power, J3 SSD1306, J4 VoiceCon, SW1 L_ENC, SW2 R_ENC, U1 6N138

Commit message: Initial work on BitBug
Other:
- net class Default removed
